File: KiCad/programador.kicad_pcb (KiCad board)
At the start: 2 copper layers, 38.4 x 16.8 mm, 24 parts, among them J1 USB_C_Receptacle, J2 Select 3.3/5V, J3 Out to mC, Q1 S8050, Q2 S8050, U1 FT232RL

Commit message: update
Parts:
- turned D3 to 180 degrees
- renumbered C1 to C4, R3 to R1, R8 to R11, R1 to R3, R6 to R5, R7 to R6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
Connections:
- net Net-(J3-Pad3) renamed /tx_+
- net Net-(J3-Pad4) renamed /rx_-
- D3 pad 1: +5V -> Net-(D3-Pad1)
- D3 pad 2: Net-(D3-Pad1) -> +5V
Routing:
- net /tx_+: track 20.2 -> 17.8 mm
